File: schema/ham-relay.sch (KiCad schematic (older format))
At the start: 62 parts, among them P1 CONN_01X08, P2 RESET, P3 ISP, P4 CONN_01X03, P5 JTAG, U1 CPC1017N, U2 XYZ, U3 REG 3V3, U4 XYZ, U5 TBB1458, U6 LPC1114FN28/102

Commit message: Update schematics
Parts:
- added TP1, TP10, TP2, TP3, TP4, TP5, TP6, TP7, TP8, TP9: TESTPOINT, Measurement_Points:Measurement_Point_Round-SMD-Pad_Small, symbol TESTPOINT
- U5: symbol OP275 -> OP275-RESCUE-ham-relay
Connections:
- net labels removed: MOD_OUT
- wire segments 146 -> 192

Commit message: Add status LED on schematics
Parts:
- added D6: STATUS, LEDs:LED-5MM, symbol LED
- added R29: 560, Resistors_ThroughHole:Resistor_Horizontal_RM10mm, symbol R
Connections:
- wire segments 192 -> 151
- no-connect marks 19 -> 18
Changed lines of the file:
@@
 $EndComp
 Wire Wire Line
-	4500 1600 4700 1600
-Wire Wire Line
-	4700 1600 4850 1600
+	4500 1600 4850 1600
 Wire Wire Line
 	4850 1900 4700 1900
 Wire Wire Line
-	4500 2550 4700 2550
-Wire Wire Line
-	4700 2550 4850 2550
+	4500 2550 4850 2550
 Wire Wire Line
 	4850 2850 4700 2850
@@
 	8100 1600 8400 1600
 Wire Wire Line
-	8400 1350 8400 1600
-Wire Wire Line
-	8400 1600 8400 1700
+	8400 1350 8400 1700
 Wire Wire Line
 	8100 1350 8400 1350
@@
 	7250 1550 7250 1600
 Wire Wire Line
-	7250 1600 7400 1600
-Wire Wire Line
-	7400 1600 8000 1600
+	7250 1600 8000 1600
 Wire Wire Line
 	7250 1450 7250 1350
 Wire Wire Line
-	7250 1350 7700 1350
-Wire Wire Line
-	7700 1350 8000 1350
+	7250 1350 8000 1350
 $Comp
 L R R23
@@
 Connection ~ 7700 1350
 Wire Wire Line
-	7250 3050 8150 3050
-Wire Wire Line
-	8850 2050 8850 2250
-Wire Wire Line
-	8850 2250 8850 3250
+	8850 2050 8850 3250
 Wire Wire Line
 	8850 2250 9550 2250
@@
 	10850 2050 10950 2050
 Wire Wire Line
-	10950 2050 10950 2150
-Wire Wire Line
-	10950 2150 10950 2250
-Wire Wire Line
-	10950 2250 10950 2350
-Wire Wire Line
-	10950 2350 10950 2450
-Wire Wire Line
-	10950 2450 10950 2550
-Wire Wire Line
-	10950 2550 10950 2650
-Wire Wire Line
-	10950 2650 10950 2750
-Wire Wire Line
-	10950 2750 10950 2850
-Wire Wire Line
-	10950 2850 10950 3050
+	10950 2050 10950 3050
 Wire Wire Line
 	10850 2150 10950 2150
@@
 	8950 2650 8950 2350
 Wire Wire Line
-	8950 2350 9050 2350
-Wire Wire Line
-	9050 2350 9550 2350
+	8950 2350 9550 2350
 Wire Wire Line
 	7250 2550 9550 2550
@@
 Wire Wire Line
 	1800 2350 1800 2450
-Wire Wire Line
-	1100 2050 1200 2050
-Wire Wire Line
-	1200 2050 1500 2050
-Wire Wire Line
-	1500 2050 1800 2050
-Wire Wire Line
-	1800 2050 2200 2050
-Wire Wire Line
-	2200 2050 2750 2050
 Connection ~ 1200 2050
 Connection ~ 1500 2050
@@
 	1200 2350 1200 2400
 Wire Wire Line
-	1500 1950 1500 2050
+	1500 2050 1500 1950
 $Comp
 L R R8
@@
 $EndComp
 Wire Wire Line
-	2100 2400 2200 2400
-Wire Wire Line
-	2200 2400 2450 2400
-Wire Wire Line
-	2200 2350 2200 2400
-Wire Wire Line
-	2200 2400 2200 2500
+	2100 2400 2450 2400
+Wire Wire Line
+	2200 2350 2200 2500
 Connection ~ 2200 2400
 Wire Wire Line
@@
 Connection ~ 2200 2050
 Wire Wire Line
-	2750 2050 2750 2350
-Wire Wire Line
 	2750 2650 2750 2900
 $Comp
@@
 $EndComp
 Wire Wire Line
-	3550 1950 3550 2050
-Wire Wire Line
-	3550 2050 3550 2350
+	3550 1950 3550 2350
 Wire Wire Line
 	3550 2650 3550 2900
@@
 $EndComp
 Wire Wire Line
-	2050 4450 2050 4200
-Wire Wire Line
-	2050 4200 2050 4050
+	2050 4050 2050 4450
 Text Label 2050 4150 2    50   ~ 0
 TONE
@@
 	2100 5400 2100 5500
 Wire Wire Line
-	2050 4950 2100 4950
-Wire Wire Line
-	2100 4950 2200 4950
+	2050 4950 2200 4950
 $Comp
 L R R5
@@
 	2550 5400 2550 5500
 Wire Wire Line
-	2500 4950 2550 4950
-Wire Wire Line
-	2550 4950 2600 4950
+	2500 4950 2600 4950
 Wire Wire Line
 	2550 4950 2550 5100
@@
 	2950 5400 2950 5500
 Wire Wire Line
-	2900 4950 2950 4950
-Wire Wire Line
-	2950 4950 3000 4950
+	2900 4950 3000 4950
 Wire Wire Line
 	2950 4950 2950 5100
@@
 	3350 5400 3350 5500
 Wire Wire Line
-	3300 4950 3350 4950
-Wire Wire Line
-	3350 4950 3750 4950
+	3300 4950 3750 4950
 Wire Wire Line
 	3350 4950 3350 5100
@@
 $EndComp
 Wire Wire Line
-	4500 5200 4550 5200
-Wire Wire Line
-	4550 5200 4600 5200
+	4500 5200 4600 5200
 $Comp
 L R R17
@@
 $EndComp
 Wire Wire Line
-	5300 5100 5350 5100
-Wire Wire Line
-	5350 5100 5400 5100
+	5300 5100 5400 5100
 Wire Wire Line
 	5350 5750 5350 5100
 Connection ~ 5350 5100
 Wire Wire Line
-	3000 6200 3450 6200
-Wire Wire Line
-	3450 6200 3750 6200
+	3000 6200 3750 6200
 $Comp
 L POT RV2
@@
 $EndComp
 Wire Wire Line
-	4500 6450 4550 6450
-Wire Wire Line
-	4550 6450 4600 6450
+	4500 6450 4600 6450
 $Comp
 L R R18
@@
 $EndComp
 Wire Wire Line
-	5300 6350 5350 6350
-Wire Wire Line
-	5350 6350 5400 6350
+	5300 6350 5400 6350
 Wire Wire Line
 	5350 7000 5350 6350
@@
 AUDIO_IN
 Wire Wire Line
-	5700 5100 5800 5100
-Wire Wire Line
-	5800 5100 5900 5100
+	5700 5100 5900 5100
 Wire Wire Line
 	5700 6350 5800 6350
@@
 	6250 5250 6250 5100
 Wire Wire Line
-	6200 5100 6250 5100
-Wire Wire Line
-	6250 5100 6450 5100
-Wire Wire Line
-	6450 5100 6900 5100
+	6200 5100 6900 5100
 Connection ~ 6250 5100
 Text Label 6900 5100 2    50   ~ 0
@@
 $EndComp
 Wire Wire Line
-	7400 5400 7750 5400
-Wire Wire Line
-	7750 5400 8150 5400
-Wire Wire Line
-	8150 5400 8200 5400
+	7400 5400 8200 5400
 Connection ~ 8150 5400
 Text Label 7400 5400 0    50   ~ 0
@@
 NoConn ~ 8800 5200
 Wire Wire Line
-	8800 5300 9050 5300
-Wire Wire Line
-	9050 5300 9100 5300
+	8800 5300 9100 5300
 Wire Wire Line
 	7250 1900 7600 1900
@@
 	9800 5200 9800 5150
 Wire Wire Line
-	9800 4600 9800 4750
-Wire Wire Line
-	9800 4750 9800 4850
+	9800 4600 9800 4850
 Text Label 9800 4700 0    50   ~ 0
 TXE
@@
 	9600 4850 9600 4750
 Wire Wire Line
-	9600 4750 9800 4750
-Wire Wire Line
-	9800 4750 10050 4750
+	9600 4750 10050 4750
 Connection ~ 9800 4750
 $Comp
@@
 NoConn ~ 10450 5200
 Wire Wire Line
-	10450 5300 10650 5300
-Wire Wire Line
-	10650 5300 11050 5300
+	10450 5300 11050 5300
 $Comp
 L C C12
@@
 NoConn ~ 7250 3350
 NoConn ~ 7250 3150
-NoConn ~ 8150 3050
-NoConn ~ 7250 2850
 NoConn ~ 7250 1650
 NoConn ~ 7250 1750
@@
 $EndComp
 Wire Wire Line
-	7400 800  7550 800
-Wire Wire Line
-	7550 800  7700 800
+	7400 800  7700 800
 Connection ~ 7550 800
 $Comp
@@
 Logic
 Connection ~ 3550 2050
-Connection ~ 2750 2050
 $Comp
 L TESTPOINT TP3
@@
 Text Label 7550 2450 2    50   ~ 0
 TONE
+Wire Wire Line
+	2750 2050 2750 2350
+Connection ~ 2750 2050
+Wire Wire Line
+	1100 2050 2750 2050
+NoConn ~ 7250 3050
+$Comp
+L R R29
+U 1 1 566E92A6
+P 7800 2850
+F 0 "R29" V 7880 2850 50  0000 C CNN
+F 1 "560" V 7800 2850 50  0000 C CNN
+F 2 "Resistors_ThroughHole:Resistor_Horizontal_RM10mm" V 7730 2850 30  0001 C CNN
+F 3 "" H 7800 2850 30  0000 C CNN
+	1    7800 2850
+	0    -1   -1   0
+$EndComp
+$Comp
+L LED D6
+U 1 1 566E92AC
+P 8250 2850
+F 0 "D6" H 8250 2950 50  0000 C CNN
+F 1 "STATUS" H 8250 2750 50  0000 C CNN
+F 2 "LEDs:LED-5MM" H 8250 2850 60  0001 C CNN
+F 3 "" H 8250 2850 60  0000 C CNN
+	1    8250 2850
+	-1   0    0    1
+$EndComp
+Wire Wire Line
+	7950 2850 8050 2850
+$Comp
+L GND #PWR058
+U 1 1 566E92B3
+P 8450 2850
+F 0 "#PWR058" H 8450 2600 50  0001 C CNN
+F 1 "GND" H 8450 2700 50  0000 C CNN
+F 2 "" H 8450 2850 60  0000 C CNN
+F 3 "" H 8450 2850 60  0000 C CNN
+	1    8450 2850
+	1    0    0    -1
+$EndComp
+Wire Wire Line
+	7650 2850 7250 2850
 $EndSCHEMATC

Commit message: First routing
Parts:
- removed C10, C15, C6, C9: 10µF, Capacitors_ThroughHole:C_Radial_D5_L6_P2.5, symbol CP
- removed C11, C8: 1µF, Capacitors_ThroughHole:C_Radial_D5_L6_P2.5, symbol CP
- removed C3: 10nF, Capacitors_ThroughHole:C_Radial_D5_L6_P2.5, symbol C
- removed C4: 330nF, Capacitors_ThroughHole:C_Radial_D5_L6_P2.5, symbol C
- removed C5: 100nF, Capacitors_ThroughHole:C_Radial_D5_L6_P2.5, symbol C
- removed C7: 47nF, Capacitors_ThroughHole:C_Radial_D5_L6_P2.5, symbol C
- removed D4: 3V3, LEDs:LED-5MM, symbol LED
- removed P5: JTAG, Pin_Headers:Pin_Header_Straight_2x10, symbol JTAG
- removed R10: 5k6, Resistors_ThroughHole:Resistor_Horizontal_RM10mm, symbol R
- removed R12, R21: 1k8, Resistors_ThroughHole:Resistor_Horizontal_RM10mm, symbol R
- removed R14, R15, R9: 47k, Resistors_ThroughHole:Resistor_Horizontal_RM10mm, symbol R
- removed R16: ?, Resistors_ThroughHole:Resistor_Horizontal_RM10mm, symbol R
- removed R17, R18: 220k, Resistors_ThroughHole:Resistor_Horizontal_RM10mm, symbol R
- removed R19, R20: 1k2, Resistors_ThroughHole:Resistor_Horizontal_RM10mm, symbol R
- removed R26, R27, R28: 10k, Resistors_ThroughHole:Resistor_Horizontal_RM10mm, symbol R
- removed RV1: 22k, Potentiometers:Potentiometer_Bourns_3005_Angular_ScrewFront, symbol POT
- removed RV2: 1k, Potentiometers:Potentiometer_Bourns_3005_Angular_ScrewFront, symbol POT
- removed TP1, TP10, TP2, TP3, TP4, TP5, TP6, TP7, TP8, TP9: TESTPOINT, Measurement_Points:Measurement_Point_Round-SMD-Pad_Small, symbol TESTPOINT
- removed U3: REG 3V3, TO_SOT_Packages_THT:TO-220_Neutral123_Vertical, symbol 7805
- removed U5: TBB1458, Housings_DIP:DIP-8_W7.62mm, symbol OP275-RESCUE-ham-relay
- added C2: 10nF, Capacitors_ThroughHole:C_Radial_D5_L6_P2.5, symbol C
- added C3: 10µF, Capacitors_ThroughHole:C_Radial_D5_L6_P2.5, symbol CP
- added C4, C5: 1µF, Capacitors_ThroughHole:C_Radial_D5_L6_P2.5, symbol CP
- added D1: 12V, LEDs:LED-5MM, symbol LED
- added IC1: 74HC126N, 74xx-eu-DIL14, symbol 74HC126N
- added J1: DB9, w_conn_d-sub:DB_9F, symbol DB9
- added P1: JTAG, Pin_Headers:Pin_Header_Straight_2x10, symbol JTAG
- added R1, R3, R4: 10k, Resistors_ThroughHole:Resistor_Horizontal_RM10mm, symbol R
- added U1: REG 3V3, TO_SOT_Packages_THT:TO-220_Neutral123_Horizontal, symbol LD1117S33TR
- D2: value 12V -> 3V3
- F1: footprint Fuse_Holders_and_Fuses:Fuseholder5x20_horiz_SemiClosed_Casing10x25mm -> Fuse_5x20mm_Holder:Fuse_5x20mm_Holder
- R5: value 680 -> ?
- R6: value ? -> 47k
- R7: value 1k8 -> 47k
- R8: value 47k -> ?
- renumbered C13 to C6, C14 to C7, C2 to C8, C12 to C9, D5 to D3, D1 to D4, D3 to D5, P1 to P2, P2 to P3, P3 to P4, P4 to P5, R1 to R10, R4 to R11, R22 to R12, R23 to R13, R2 to R14, R3 to R15, R11 to R16, R29 to R17, R13 to R18, R25 to R2, R24 to R9, U6 to U2, U1 to U3, U2 to U4, U4 to U5
Connections:
- net labels added: ISP, RESET, SWCLK, SWDIO, SWO, TONE_OUT
- net labels removed: AUDIO_IN, AUDIO_OUT
- wire segments 151 -> 132
- no-connect marks 18 -> 19
Other:
- note added: "SWD"
- note removed: "Audio"
- note removed: "Logic"
- moved on the sheet: C6, C7, C8, C9, D3, D4, D5, D6, P2, P3, P4, P5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

Commit message: Update schematic
Parts:
- renumbered IC1 to U7
Changed lines of the file:
@@
 Title "Logique relais"
 Date "2015-12-21"
-Rev "4"
+Rev "5"
 Comp ""
 Comment1 ""
@@
 NoConn ~ 6250 2250
 $Comp
-L 74HC126N IC1
+L 74HC126N U7
 U 1 1 567894D6
 P 8600 1350
-F 0 "IC1" H 8700 1475 50  0000 L BNN
+F 0 "U7" H 8700 1475 50  0000 L BNN
 F 1 "74HC126N" H 8700 1150 50  0000 L BNN
 F 2 "Housings_DIP:DIP-14_W7.62mm" H 8600 1500 50  0001 C CNN
@@
 $EndComp
 $Comp
-L 74HC126N IC1
+L 74HC126N U7
 U 2 1 56789565
 P 8600 2100
-F 0 "IC1" H 8700 2225 50  0000 L BNN
+F 0 "U7" H 8700 2225 50  0000 L BNN
 F 1 "74HC126N" H 8700 1900 50  0000 L BNN
 F 2 "Housings_DIP:DIP-14_W7.62mm" H 8600 2250 50  0001 C CNN
@@
 $EndComp
 $Comp
-L 74HC126N IC1
+L 74HC126N U7
 U 3 1 567895EA
 P 8600 2850
-F 0 "IC1" H 8700 2975 50  0000 L BNN
+F 0 "U7" H 8700 2975 50  0000 L BNN
 F 1 "74HC126N" H 8700 2650 50  0000 L BNN
 F 2 "Housings_DIP:DIP-14_W7.62mm" H 8600 3000 50  0001 C CNN
@@
 $EndComp
 $Comp
-L 74HC126N IC1
+L 74HC126N U7
 U 5 1 5678965D
 P 8500 3750
-F 0 "IC1" H 8600 3875 50  0000 L BNN
+F 0 "U7" H 8600 3875 50  0000 L BNN
 F 1 "74HC126N" H 8600 3550 50  0000 L BNN
 F 2 "Housings_DIP:DIP-14_W7.62mm" H 8500 3900 50  0001 C CNN
@@
 $EndComp
 $Comp
-L 74HC126N IC1
+L 74HC126N U7
 U 4 1 56781E99
 P 9600 3700
-F 0 "IC1" H 9700 3825 50  0000 L BNN
+F 0 "U7" H 9700 3825 50  0000 L BNN
 F 1 "74HC126N" H 9700 3500 50  0000 L BNN
 F 2 "74xx-eu-DIL14" H 9600 3850 50  0001 C CNN

Commit message: More changes
Parts:
- removed C4: 1µF, Capacitors_ThroughHole:C_Radial_D5_L6_P2.5, symbol CP
- removed U1: REG 3V3, TO_SOT_Packages_THT:TO-220_Neutral123_Horizontal, symbol LD1117S33TR
- added U1: REG3V3, TO_SOT_Packages_THT:TO-220_Neutral123_Horizontal, symbol 7805
- C1, C3, C5: footprint Capacitors_ThroughHole:C_Radial_D5_L6_P2.5 -> Capacitors_ThroughHole:C_Radial_D5_L11_P2.5
- C2, C6, C7, C8, C9: footprint Capacitors_ThroughHole:C_Radial_D5_L6_P2.5 -> Capacitors_ThroughHole:C_Rect_L4_W2.5_P2.5
- D1, D2, D3, D4, D5, D6: footprint LEDs:LED-5MM -> LEDs:LED-3MM
- F1: footprint Fuse_5x20mm_Holder:Fuse_5x20mm_Holder -> Fuse_Holders_and_Fuses:Fuseholder5x20_horiz_open_lateral_Type-II
- R1, R10, R11, R12, R13, R14, R15, R16, R17, R18, R2, R3, R4, R5, R6, R7, R8, R9: footprint Resistors_ThroughHole:Resistor_Horizontal_RM10mm -> resistors:Resistor_Horizontal_RM08mm
- U3: Mouser (none) -> 782-LH1540AT
- U7: footprint 74xx-eu-DIL14 -> Housings_DIP:DIP-14_W7.62mm
Connections:
- wire segments 132 -> 130
Other:
- moved on the sheet: C5, D2, R8

Commit message: Update footprints
Parts:
- C2, C6, C7, C8, C9: footprint Capacitors_ThroughHole:C_Rect_L4_W2.5_P2.5 -> Capacitors_ThroughHole:C_Rect_L7_W2.5_P5
- F1: footprint Fuse_Holders_and_Fuses:Fuseholder5x20_horiz_open_lateral_Type-II -> Fuse_Holders_and_Fuses:Fuseholder5x20_horiz_SemiClosed_Casing10x25mm
Changed lines of the file:
@@
 F 0 "C6" H 3725 1850 50  0000 L CNN
 F 1 "100nF" H 3725 1650 50  0000 L CNN
-F 2 "Capacitors_ThroughHole:C_Rect_L4_W2.5_P2.5" H 3738 1600 30  0001 C CNN
+F 2 "Capacitors_ThroughHole:C_Rect_L7_W2.5_P5" H 3738 1600 30  0001 C CNN
 F 3 "" H 3700 1750 60  0000 C CNN
 	1    3700 1750
@@
 F 0 "C7" H 3725 2800 50  0000 L CNN
 F 1 "100nF" H 3725 2600 50  0000 L CNN
-F 2 "Capacitors_ThroughHole:C_Rect_L4_W2.5_P2.5" H 3738 2550 30  0001 C CNN
+F 2 "Capacitors_ThroughHole:C_Rect_L7_W2.5_P5" H 3738 2550 30  0001 C CNN
 F 3 "" H 3700 2700 60  0000 C CNN
 	1    3700 2700
@@
 F 0 "C8" H 8075 5650 50  0000 L CNN
 F 1 "10nF" H 8075 5450 50  0000 L CNN
-F 2 "Capacitors_ThroughHole:C_Rect_L4_W2.5_P2.5" H 8088 5400 30  0001 C CNN
+F 2 "Capacitors_ThroughHole:C_Rect_L7_W2.5_P5" H 8088 5400 30  0001 C CNN
 F 3 "" H 8050 5550 60  0000 C CNN
 	1    8050 5550
@@
 F 0 "C9" H 10525 5550 50  0000 L CNN
 F 1 "10nF" H 10525 5350 50  0000 L CNN
-F 2 "Capacitors_ThroughHole:C_Rect_L4_W2.5_P2.5" H 10538 5300 30  0001 C CNN
+F 2 "Capacitors_ThroughHole:C_Rect_L7_W2.5_P5" H 10538 5300 30  0001 C CNN
 F 3 "" H 10500 5450 60  0000 C CNN
 	1    10500 5450
@@
 F 0 "F1" H 1250 6200 50  0000 C CNN
 F 1 "FUSE" H 1050 6100 50  0000 C CNN
-F 2 "Fuse_Holders_and_Fuses:Fuseholder5x20_horiz_open_lateral_Type-II" H 1150 6150 60  0001 C CNN
+F 2 "Fuse_Holders_and_Fuses:Fuseholder5x20_horiz_SemiClosed_Casing10x25mm" H 1150 6150 60  0001 C CNN
 F 3 "" H 1150 6150 60  0000 C CNN
 	1    1150 6150
@@
 F 0 "C2" H 1575 6650 50  0000 L CNN
 F 1 "10nF" H 1575 6450 50  0000 L CNN
-F 2 "Capacitors_ThroughHole:C_Rect_L4_W2.5_P2.5" H 1588 6400 30  0001 C CNN
+F 2 "Capacitors_ThroughHole:C_Rect_L7_W2.5_P5" H 1588 6400 30  0001 C CNN
 F 3 "" H 1550 6550 60  0000 C CNN
 	1    1550 6550

Commit message: Add EXT_CR support
Parts:
- added C4: 10nF, Capacitors_ThroughHole:C_Rect_L7_W2.5_P5, symbol C
- added R31: ?, resistors:Resistor_Horizontal_RM08mm, symbol R
- added U8: XYZ, Housings_DIP:DIP-6_W7.62mm, symbol CNY17-1
Connections:
- net Audio/AUDIO_IN: now also P2.5 (P5); no longer P2.4 (P4)
- net Audio/AUDIO_OUT: now also P2.6 (P6); no longer P2.5 (P5)
- net GND: now also C4.2, U8.4
- net VCC: now also R31.1
- net EXT: now reaches U2.26 (PIO0_3)
- net EXT: now also U8.5
- new net: R31.2, U8.1
- new net EXT_CR: C4.1, P2.4 (P4), U8.2
- no-connect marks 19 -> 18
Other:
- moved on the sheet: C8, D3, D4, P2, R10, R11, R12, R13, R14, R15, R9, U3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

Commit message: Component placement
Parts:
- renumbered C5 to C4, C6 to C5, C7 to C6, C4 to C7, D3 to D2, D2 to D3, R8 to R10, R31 to R12, R12 to R13, R13 to R14, R14 to R15, R15 to R16, R16 to R17, R17 to R18, R18 to R19, R9 to R8, R10 to R9, U3 to U2, U2 to U3, U8 to U4, U4 to U5, U7 to U6, U5 to U7
Connections:
- net Audio/AUDIO_OUT: now also P2.7 (P7); no longer P2.6 (P6)
- net GND: now also P2.6 (P6)
- no-connect marks 18 -> 17
