File: schema/ham-relay.sch (KiCad schematic (older format))
At the start: 52 parts, among them J1 DB9, P1 JTAG, P2 CONN_01X08, P3 RESET, P4 ISP, P5 CONN_01X03, U1 REG3V3, U2 CPC1017N, U3 LPC1114FN28/102, U4 MCA231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

Commit message: Update schematics after prototype validation
Parts:
- removed U2: CPC1017N, Housings_DIP:DIP-6_W7.62mm, symbol CPC1017N
- added U2: LH1540, symbol LH1540
- R33, R34: value 560k -> 56k
Connections:
- wire segments 141 -> 143
Other:
- moved on the sheet: R11
Changed lines of the file:
@@
 Sheet 1 2
 Title "Logique relais"
-Date "2016-04-08"
+Date "2016-04-09"
 Rev "7"
 Comp ""
@@
 Wire Wire Line
 	3500 2550 3500 1600
-$Comp
-L CPC1017N U2
-U 1 1 5664A880
-P 3900 5050
-F 0 "U2" H 3900 5400 60  0000 C CNN
-F 1 "CPC1017N" H 3900 4693 60  0000 C CNN
-F 2 "Housings_DIP:DIP-6_W7.62mm" H 3900 5050 60  0001 C CNN
-F 3 "" H 3900 5050 60  0000 C CNN
-F 4 "782-LH1540AT" H 3900 5050 60  0001 C CNN "Mouser"
-	1    3900 5050
-	1    0    0    -1
-$EndComp
-Wire Wire Line
-	4800 4800 4300 4800
-Text Label 4800 4800 2    50   ~ 0
+Text Label 4600 4950 2    50   ~ 0
 TONE
 $Comp
@@
 $EndComp
 Wire Wire Line
-	3500 5200 3500 5250
+	3500 5150 3500 5250
 $Comp
 L R R9
@@
 	3500 4150 3500 4550
 Wire Wire Line
-	3500 4850 3500 4900
+	3500 4850 3500 4950
 $Comp
 L R R8
@@
 L R R11
 U 1 1 56651136
-P 4350 5600
-F 0 "R11" V 4430 5600 50  0000 C CNN
-F 1 "2k2" V 4350 5600 50  0000 C CNN
-F 2 "resistors:Resistor_Horizontal_RM08mm" V 4280 5600 30  0001 C CNN
-F 3 "" H 4350 5600 30  0000 C CNN
-	1    4350 5600
+P 4200 5450
+F 0 "R11" V 4280 5450 50  0000 C CNN
+F 1 "2k2" V 4200 5450 50  0000 C CNN
+F 2 "resistors:Resistor_Horizontal_RM08mm" V 4130 5450 30  0001 C CNN
+F 3 "" H 4200 5450 30  0000 C CNN
+	1    4200 5450
 	1    0    0    -1
 $EndComp
@@
 L GND #PWR07
 U 1 1 5665113C
-P 4350 5850
-F 0 "#PWR07" H 4350 5600 50  0001 C CNN
-F 1 "GND" H 4350 5700 50  0000 C CNN
-F 2 "" H 4350 5850 60  0000 C CNN
-F 3 "" H 4350 5850 60  0000 C CNN
-	1    4350 5850
-	1    0    0    -1
-$EndComp
-Wire Wire Line
-	4350 5300 4350 5450
-Wire Wire Line
-	4350 5750 4350 5850
-Wire Wire Line
-	4300 5300 4800 5300
-Connection ~ 4350 5300
+P 4200 5700
+F 0 "#PWR07" H 4200 5450 50  0001 C CNN
+F 1 "GND" H 4200 5550 50  0000 C CNN
+F 2 "" H 4200 5700 60  0000 C CNN
+F 3 "" H 4200 5700 60  0000 C CNN
+	1    4200 5700
+	1    0    0    -1
+$EndComp
+Wire Wire Line
+	4200 5150 4200 5300
+Wire Wire Line
+	4200 5600 4200 5700
+Connection ~ 4200 5150
 $Comp
 L CONN_01X08 P2
@@
 F4 "TONE" I L 5450 7300 50
 $EndSheet
-Text Label 4800 5300 2    50   ~ 0
+Text Label 4600 5150 2    50   ~ 0
 TONE_OUT
 $Comp
@@
 P 7350 1300
 F 0 "R34" V 7430 1300 50  0000 C CNN
-F 1 "560k" V 7350 1300 50  0000 C CNN
+F 1 "56k" V 7350 1300 50  0000 C CNN
 F 2 "resistors:Resistor_Horizontal_RM08mm" V 7280 1300 30  0001 C CNN
 F 3 "" H 7350 1300 30  0000 C CNN
@@
 P 7050 1750
 F 0 "R33" V 7130 1750 50  0000 C CNN
-F 1 "560k" V 7050 1750 50  0000 C CNN
+F 1 "56k" V 7050 1750 50  0000 C CNN
 F 2 "resistors:Resistor_Horizontal_RM08mm" V 6980 1750 30  0001 C CNN
 F 3 "" H 7050 1750 30  0000 C CNN
@@
 Connection ~ 7050 1900
 Connection ~ 7650 1300
+$Comp
+L LH1540 U2
+U 1 1 57095F3F
+P 3850 5050
+F 0 "U2" H 3650 5250 50  0000 L CNN
+F 1 "LH1540" H 3850 5250 50  0000 L CNN
+F 2 "" H 3650 4850 50  0000 L CIN
+F 3 "" H 3800 5050 50  0000 L CNN
+	1    3850 5050
+	1    0    0    -1
+$EndComp
+Wire Wire Line
+	3500 4950 3550 4950
+Wire Wire Line
+	3550 5150 3500 5150
+Wire Wire Line
+	4150 4950 4600 4950
+Wire Wire Line
+	4150 5150 4600 5150
 $EndSCHEMATC
