File: schema/audio.sch (KiCad schematic (older format))
At the start: 20 parts, among them U6 TBB1458

Commit message: Update schematic
Parts:
- added R30: 22k, Resistors_ThroughHole:Resistor_Horizontal_RM10mm, symbol R
- C12: value 47nF -> 33nF
- R19: value 680 -> 560
- RV1: value 22k -> 10k
Connections:
- wire segments 37 -> 38
Other:
- moved on the sheet: C10, C11, C12, R19, R20, R21
Changed lines of the file:
@@
 Title "Logique relais"
 Date "2015-12-21"
-Rev "4"
+Rev "5"
 Comp ""
 Comment1 ""
@@
 $EndDescr
 Wire Wire Line
-	2700 2100 2850 2100
+	2650 2100 2800 2100
 $Comp
 L R R19
 U 1 1 5677F0F1
-P 3000 2100
-F 0 "R19" V 3080 2100 50  0000 C CNN
-F 1 "680" V 3000 2100 50  0000 C CNN
-F 2 "Resistors_ThroughHole:Resistor_Horizontal_RM10mm" V 2930 2100 30  0001 C CNN
-F 3 "" H 3000 2100 30  0000 C CNN
-	1    3000 2100
+P 2950 2100
+F 0 "R19" V 3030 2100 50  0000 C CNN
+F 1 "560" V 2950 2100 50  0000 C CNN
+F 2 "Resistors_ThroughHole:Resistor_Horizontal_RM10mm" V 2880 2100 30  0001 C CNN
+F 3 "" H 2950 2100 30  0000 C CNN
+	1    2950 2100
 	0    1    1    0
 $EndComp
@@
 L C C10
 U 1 1 5677F0F8
-P 3200 2400
-F 0 "C10" H 3225 2500 50  0000 L CNN
-F 1 "330nF" H 3225 2300 50  0000 L CNN
-F 2 "Capacitors_ThroughHole:C_Radial_D5_L6_P2.5" H 3238 2250 30  0001 C CNN
-F 3 "" H 3200 2400 60  0000 C CNN
-	1    3200 2400
+P 3150 2400
+F 0 "C10" H 3175 2500 50  0000 L CNN
+F 1 "330nF" H 3175 2300 50  0000 L CNN
+F 2 "Capacitors_ThroughHole:C_Radial_D5_L6_P2.5" H 3188 2250 30  0001 C CNN
+F 3 "" H 3150 2400 60  0000 C CNN
+	1    3150 2400
 	1    0    0    -1
 $EndComp
@@
 L GND #PWR51
 U 1 1 5677F0FF
-P 3200 2650
-F 0 "#PWR51" H 3200 2400 50  0001 C CNN
-F 1 "GND" H 3200 2500 50  0000 C CNN
-F 2 "" H 3200 2650 60  0000 C CNN
-F 3 "" H 3200 2650 60  0000 C CNN
-	1    3200 2650
-	1    0    0    -1
-$EndComp
-Wire Wire Line
-	3200 2550 3200 2650
-Wire Wire Line
-	3150 2100 3250 2100
-Wire Wire Line
-	3200 2100 3200 2250
+P 3150 2650
+F 0 "#PWR51" H 3150 2400 50  0001 C CNN
+F 1 "GND" H 3150 2500 50  0000 C CNN
+F 2 "" H 3150 2650 60  0000 C CNN
+F 3 "" H 3150 2650 60  0000 C CNN
+	1    3150 2650
+	1    0    0    -1
+$EndComp
+Wire Wire Line
+	3150 2550 3150 2650
+Wire Wire Line
+	3100 2100 3200 2100
+Wire Wire Line
+	3150 2100 3150 2250
 $Comp
 L R R20
 U 1 1 5677F108
-P 3400 2100
-F 0 "R20" V 3480 2100 50  0000 C CNN
-F 1 "1k8" V 3400 2100 50  0000 C CNN
-F 2 "Resistors_ThroughHole:Resistor_Horizontal_RM10mm" V 3330 2100 30  0001 C CNN
-F 3 "" H 3400 2100 30  0000 C CNN
-	1    3400 2100
+P 3350 2100
+F 0 "R20" V 3430 2100 50  0000 C CNN
+F 1 "1k8" V 3350 2100 50  0000 C CNN
+F 2 "Resistors_ThroughHole:Resistor_Horizontal_RM10mm" V 3280 2100 30  0001 C CNN
+F 3 "" H 3350 2100 30  0000 C CNN
+	1    3350 2100
 	0    1    1    0
 $EndComp
@@
 L C C11
 U 1 1 5677F10F
-P 3600 2400
-F 0 "C11" H 3625 2500 50  0000 L CNN
-F 1 "100nF" H 3625 2300 50  0000 L CNN
-F 2 "Capacitors_ThroughHole:C_Radial_D5_L6_P2.5" H 3638 2250 30  0001 C CNN
-F 3 "" H 3600 2400 60  0000 C CNN
-	1    3600 2400
+P 3550 2400
+F 0 "C11" H 3575 2500 50  0000 L CNN
+F 1 "100nF" H 3575 2300 50  0000 L CNN
+F 2 "Capacitors_ThroughHole:C_Radial_D5_L6_P2.5" H 3588 2250 30  0001 C CNN
+F 3 "" H 3550 2400 60  0000 C CNN
+	1    3550 2400
 	1    0    0    -1
 $EndComp
@@
 L GND #PWR52
 U 1 1 5677F116
-P 3600 2650
-F 0 "#PWR52" H 3600 2400 50  0001 C CNN
-F 1 "GND" H 3600 2500 50  0000 C CNN
-F 2 "" H 3600 2650 60  0000 C CNN
-F 3 "" H 3600 2650 60  0000 C CNN
-	1    3600 2650
-	1    0    0    -1
-$EndComp
-Wire Wire Line
-	3600 2550 3600 2650
-Wire Wire Line
-	3550 2100 3650 2100
-Wire Wire Line
-	3600 2100 3600 2250
+P 3550 2650
+F 0 "#PWR52" H 3550 2400 50  0001 C CNN
+F 1 "GND" H 3550 2500 50  0000 C CNN
+F 2 "" H 3550 2650 60  0000 C CNN
+F 3 "" H 3550 2650 60  0000 C CNN
+	1    3550 2650
+	1    0    0    -1
+$EndComp
+Wire Wire Line
+	3550 2550 3550 2650
+Wire Wire Line
+	3500 2100 3600 2100
+Wire Wire Line
+	3550 2100 3550 2250
 $Comp
 L R R21
 U 1 1 5677F11F
-P 3800 2100
-F 0 "R21" V 3880 2100 50  0000 C CNN
-F 1 "5k6" V 3800 2100 50  0000 C CNN
-F 2 "Resistors_ThroughHole:Resistor_Horizontal_RM10mm" V 3730 2100 30  0001 C CNN
-F 3 "" H 3800 2100 30  0000 C CNN
-	1    3800 2100
+P 3750 2100
+F 0 "R21" V 3830 2100 50  0000 C CNN
+F 1 "5k6" V 3750 2100 50  0000 C CNN
+F 2 "Resistors_ThroughHole:Resistor_Horizontal_RM10mm" V 3680 2100 30  0001 C CNN
+F 3 "" H 3750 2100 30  0000 C CNN
+	1    3750 2100
 	0    1    1    0
 $EndComp
@@
 L C C12
 U 1 1 5677F126
-P 4000 2400
-F 0 "C12" H 4025 2500 50  0000 L CNN
-F 1 "47nF" H 4025 2300 50  0000 L CNN
-F 2 "Capacitors_ThroughHole:C_Radial_D5_L6_P2.5" H 4038 2250 30  0001 C CNN
-F 3 "" H 4000 2400 60  0000 C CNN
-	1    4000 2400
+P 3950 2400
+F 0 "C12" H 3975 2500 50  0000 L CNN
+F 1 "33nF" H 3975 2300 50  0000 L CNN
+F 2 "Capacitors_ThroughHole:C_Radial_D5_L6_P2.5" H 3988 2250 30  0001 C CNN
+F 3 "" H 3950 2400 60  0000 C CNN
+	1    3950 2400
 	1    0    0    -1
 $EndComp
@@
 L GND #PWR53
 U 1 1 5677F12D
-P 4000 2650
-F 0 "#PWR53" H 4000 2400 50  0001 C CNN
-F 1 "GND" H 4000 2500 50  0000 C CNN
-F 2 "" H 4000 2650 60  0000 C CNN
-F 3 "" H 4000 2650 60  0000 C CNN
-	1    4000 2650
-	1    0    0    -1
-$EndComp
-Wire Wire Line
-	4000 2550 4000 2650
-Wire Wire Line
-	3950 2100 4400 2100
-Wire Wire Line
-	4000 2100 4000 2250
-Connection ~ 3200 2100
-Connection ~ 3600 2100
+P 3950 2650
+F 0 "#PWR53" H 3950 2400 50  0001 C CNN
+F 1 "GND" H 3950 2500 50  0000 C CNN
+F 2 "" H 3950 2650 60  0000 C CNN
+F 3 "" H 3950 2650 60  0000 C CNN
+	1    3950 2650
+	1    0    0    -1
+$EndComp
+Wire Wire Line
+	3950 2550 3950 2650
+Wire Wire Line
+	3900 2100 4000 2100
+Wire Wire Line
+	3950 2100 3950 2250
+Connection ~ 3150 2100
+Connection ~ 3550 2100
 $Comp
 L POT RV1
@@
 P 4400 2350
 F 0 "RV1" H 4400 2250 50  0000 C CNN
-F 1 "22k" H 4400 2350 50  0000 C CNN
+F 1 "10k" H 4400 2350 50  0000 C CNN
 F 2 "Potentiometers:Potentiometer_Triwood_RM-065" H 4400 2350 60  0001 C CNN
 F 3 "" H 4400 2350 60  0000 C CNN
@@
 Wire Wire Line
 	4400 2600 4400 2650
-Connection ~ 4000 2100
+Connection ~ 3950 2100
 $Comp
 L CP C13
@@
 Text HLabel 3950 3350 0    50   Input ~ 0
 AUDIO_IN
-Text HLabel 2700 2100 0    50   Input ~ 0
+Text HLabel 2650 2100 0    50   Input ~ 0
 TONE
+$Comp
+L R R30
+U 1 1 567C5134
+P 4150 2100
+F 0 "R30" V 4230 2100 50  0000 C CNN
+F 1 "22k" V 4150 2100 50  0000 C CNN
+F 2 "Resistors_ThroughHole:Resistor_Horizontal_RM10mm" V 4080 2100 30  0001 C CNN
+F 3 "" H 4150 2100 30  0000 C CNN
+	1    4150 2100
+	0    1    1    0
+$EndComp
+Wire Wire Line
+	4300 2100 4400 2100
 $EndSCHEMATC

Commit message: More changes
Parts:
- C10, C11, C12: footprint Capacitors_ThroughHole:C_Radial_D5_L6_P2.5 -> Capacitors_ThroughHole:C_Rect_L7_W3.5_P5
- C13, C14, C15: footprint Capacitors_ThroughHole:C_Radial_D5_L6_P2.5 -> Capacitors_ThroughHole:C_Radial_D5_L11_P2.5
- R19, R20, R21, R22, R23, R24, R25, R26, R27, R28, R29, R30: footprint Resistors_ThroughHole:Resistor_Horizontal_RM10mm -> resistors:Resistor_Horizontal_RM08mm
- RV1: footprint Potentiometers:Potentiometer_Triwood_RM-065 -> Potentiometres:POT93YB
- RV2: footprint Potentiometers:Potentiometer_Triwood_RM-065 -> Potentiometres:POT93YA
Changed lines of the file:
@@
 LIBS:74xx-eu
 LIBS:resistor-bourns
+LIBS:7805
 LIBS:ham-relay-cache
 EELAYER 25 0
@@
 F 0 "R19" V 3030 2100 50  0000 C CNN
 F 1 "560" V 2950 2100 50  0000 C CNN
-F 2 "Resistors_ThroughHole:Resistor_Horizontal_RM10mm" V 2880 2100 30  0001 C CNN
+F 2 "resistors:Resistor_Horizontal_RM08mm" V 2880 2100 30  0001 C CNN
 F 3 "" H 2950 2100 30  0000 C CNN
 	1    2950 2100
@@
 F 0 "C10" H 3175 2500 50  0000 L CNN
 F 1 "330nF" H 3175 2300 50  0000 L CNN
-F 2 "Capacitors_ThroughHole:C_Radial_D5_L6_P2.5" H 3188 2250 30  0001 C CNN
+F 2 "Capacitors_ThroughHole:C_Rect_L7_W3.5_P5" H 3188 2250 30  0001 C CNN
 F 3 "" H 3150 2400 60  0000 C CNN
 	1    3150 2400
@@
 $EndComp
 $Comp
-L GND #PWR51
+L GND #PWR050
 U 1 1 5677F0FF
 P 3150 2650
-F 0 "#PWR51" H 3150 2400 50  0001 C CNN
+F 0 "#PWR050" H 3150 2400 50  0001 C CNN
 F 1 "GND" H 3150 2500 50  0000 C CNN
 F 2 "" H 3150 2650 60  0000 C CNN
@@
 F 0 "R20" V 3430 2100 50  0000 C CNN
 F 1 "1k8" V 3350 2100 50  0000 C CNN
-F 2 "Resistors_ThroughHole:Resistor_Horizontal_RM10mm" V 3280 2100 30  0001 C CNN
+F 2 "resistors:Resistor_Horizontal_RM08mm" V 3280 2100 30  0001 C CNN
 F 3 "" H 3350 2100 30  0000 C CNN
 	1    3350 2100
@@
 F 0 "C11" H 3575 2500 50  0000 L CNN
 F 1 "100nF" H 3575 2300 50  0000 L CNN
-F 2 "Capacitors_ThroughHole:C_Radial_D5_L6_P2.5" H 3588 2250 30  0001 C CNN
+F 2 "Capacitors_ThroughHole:C_Rect_L7_W3.5_P5" H 3588 2250 30  0001 C CNN
 F 3 "" H 3550 2400 60  0000 C CNN
 	1    3550 2400
@@
 $EndComp
 $Comp
-L GND #PWR52
+L GND #PWR051
 U 1 1 5677F116
 P 3550 2650
-F 0 "#PWR52" H 3550 2400 50  0001 C CNN
+F 0 "#PWR051" H 3550 2400 50  0001 C CNN
 F 1 "GND" H 3550 2500 50  0000 C CNN
 F 2 "" H 3550 2650 60  0000 C CNN
@@
 F 0 "R21" V 3830 2100 50  0000 C CNN
 F 1 "5k6" V 3750 2100 50  0000 C CNN
-F 2 "Resistors_ThroughHole:Resistor_Horizontal_RM10mm" V 3680 2100 30  0001 C CNN
+F 2 "resistors:Resistor_Horizontal_RM08mm" V 3680 2100 30  0001 C CNN
 F 3 "" H 3750 2100 30  0000 C CNN
 	1    3750 2100
@@
 F 0 "C12" H 3975 2500 50  0000 L CNN
 F 1 "33nF" H 3975 2300 50  0000 L CNN
-F 2 "Capacitors_ThroughHole:C_Radial_D5_L6_P2.5" H 3988 2250 30  0001 C CNN
+F 2 "Capacitors_ThroughHole:C_Rect_L7_W3.5_P5" H 3988 2250 30  0001 C CNN
 F 3 "" H 3950 2400 60  0000 C CNN
 	1    3950 2400
@@
 $EndComp
 $Comp
-L GND #PWR53
+L GND #PWR052
 U 1 1 5677F12D
 P 3950 2650
-F 0 "#PWR53" H 3950 2400 50  0001 C CNN
+F 0 "#PWR052" H 3950 2400 50  0001 C CNN
 F 1 "GND" H 3950 2500 50  0000 C CNN
 F 2 "" H 3950 2650 60  0000 C CNN
@@
 F 0 "RV1" H 4400 2250 50  0000 C CNN
 F 1 "10k" H 4400 2350 50  0000 C CNN
-F 2 "Potentiometers:Potentiometer_Triwood_RM-065" H 4400 2350 60  0001 C CNN
+F 2 "Potentiometres:POT93YB" H 4400 2350 60  0001 C CNN
 F 3 "" H 4400 2350 60  0000 C CNN
 	1    4400 2350
@@
 $EndComp
 $Comp
-L GND #PWR55
+L GND #PWR053
 U 1 1 5677F13F
 P 4400 2650
-F 0 "#PWR55" H 4400 2400 50  0001 C CNN
+F 0 "#PWR053" H 4400 2400 50  0001 C CNN
 F 1 "GND" H 4400 2500 50  0000 C CNN
 F 2 "" H 4400 2650 60  0000 C CNN
@@
 F 0 "C13" H 4725 2450 50  0000 L CNN
 F 1 "10µF" H 4725 2250 50  0000 L CNN
-F 2 "Capacitors_ThroughHole:C_Radial_D5_L6_P2.5" H 4738 2200 30  0001 C CNN
+F 2 "Capacitors_ThroughHole:C_Radial_D5_L11_P2.5" H 4738 2200 30  0001 C CNN
 F 3 "" H 4700 2350 60  0000 C CNN
 	1    4700 2350
@@
 F 0 "R23" V 5080 2350 50  0000 C CNN
 F 1 "47k" V 5000 2350 50  0000 C CNN
-F 2 "Resistors_ThroughHole:Resistor_Horizontal_RM10mm" V 4930 2350 30  0001 C CNN
+F 2 "resistors:Resistor_Horizontal_RM08mm" V 4930 2350 30  0001 C CNN
 F 3 "" H 5000 2350 30  0000 C CNN
 	1    5000 2350
@@
 F 0 "R25" V 5680 2900 50  0000 C CNN
 F 1 "220k" V 5600 2900 50  0000 C CNN
-F 2 "Resistors_ThroughHole:Resistor_Horizontal_RM10mm" V 5530 2900 30  0001 C CNN
+F 2 "resistors:Resistor_Horizontal_RM08mm" V 5530 2900 30  0001 C CNN
 F 3 "" H 5600 2900 30  0000 C CNN
 	1    5600 2900
@@
 $EndComp
 $Comp
-L GND #PWR60
+L GND #PWR054
 U 1 1 5677F164
 P 5500 2550
-F 0 "#PWR60" H 5500 2300 50  0001 C CNN
+F 0 "#PWR054" H 5500 2300 50  0001 C CNN
 F 1 "GND" H 5500 2400 50  0000 C CNN
 F 2 "" H 5500 2550 60  0000 C CNN
@@
 F 0 "R27" V 6280 2250 50  0000 C CNN
 F 1 "1k2" V 6200 2250 50  0000 C CNN
-F 2 "Resistors_ThroughHole:Resistor_Horizontal_RM10mm" V 6130 2250 30  0001 C CNN
+F 2 "resistors:Resistor_Horizontal_RM08mm" V 6130 2250 30  0001 C CNN
 F 3 "" H 6200 2250 30  0000 C CNN
 	1    6200 2250
@@
 F 0 "RV2" H 4400 3500 50  0000 C CNN
 F 1 "1k" H 4400 3600 50  0000 C CNN
-F 2 "Potentiometers:Potentiometer_Triwood_RM-065" H 4400 3600 60  0001 C CNN
+F 2 "Potentiometres:POT93YA" H 4400 3600 60  0001 C CNN
 F 3 "" H 4400 3600 60  0000 C CNN
 	1    4400 3600
@@
 $EndComp
 $Comp
-L GND #PWR56
+L GND #PWR055
 U 1 1 5677F180
 P 4400 3900
-F 0 "#PWR56" H 4400 3650 50  0001 C CNN
+F 0 "#PWR055" H 4400 3650 50  0001 C CNN
 F 1 "GND" H 4400 3750 50  0000 C CNN
 F 2 "" H 4400 3900 60  0000 C CNN
@@
 F 0 "C14" H 4725 3700 50  0000 L CNN
 F 1 "10µF" H 4725 3500 50  0000 L CNN
-F 2 "Capacitors_ThroughHole:C_Radial_D5_L6_P2.5" H 4738 3450 30  0001 C CNN
+F 2 "Capacitors_ThroughHole:C_Radial_D5_L11_P2.5" H 4738 3450 30  0001 C CNN
 F 3 "" H 4700 3600 60  0000 C CNN
 	1    4700 3600
@@
 F 0 "R24" V 5080 3600 50  0000 C CNN
 F 1 "47k" V 5000 3600 50  0000 C CNN
-F 2 "Resistors_ThroughHole:Resistor_Horizontal_RM10mm" V 4930 3600 30  0001 C CNN
+F 2 "resistors:Resistor_Horizontal_RM08mm" V 4930 3600 30  0001 C CNN
 F 3 "" H 5000 3600 30  0000 C CNN
 	1    5000 3600
@@
 F 0 "R26" V 5680 4150 50  0000 C CNN
 F 1 "220k" V 5600 4150 50  0000 C CNN
-F 2 "Resistors_ThroughHole:Resistor_Horizontal_RM10mm" V 5530 4150 30  0001 C CNN
+F 2 "resistors:Resistor_Horizontal_RM08mm" V 5530 4150 30  0001 C CNN
 F 3 "" H 5600 4150 30  0000 C CNN
 	1    5600 4150
@@
 $EndComp
 $Comp
-L GND #PWR62
+L GND #PWR056
 U 1 1 5677F19D
 P 5500 3800
-F 0 "#PWR62" H 5500 3550 50  0001 C CNN
+F 0 "#PWR056" H 5500 3550 50  0001 C CNN
 F 1 "GND" H 5500 3650 50  0000 C CNN
 F 2 "" H 5500 3800 60  0000 C CNN
@@
 F 0 "R28" V 6280 3500 50  0000 C CNN
 F 1 "1k2" V 6200 3500 50  0000 C CNN
-F 2 "Resistors_ThroughHole:Resistor_Horizontal_RM10mm" V 6130 3500 30  0001 C CNN
+F 2 "resistors:Resistor_Horizontal_RM08mm" V 6130 3500 30  0001 C CNN
 F 3 "" H 6200 3500 30  0000 C CNN
 	1    6200 3500
@@
 F 0 "R22" V 4180 3650 50  0000 C CNN
 F 1 "1k8" V 4100 3650 50  0000 C CNN
-F 2 "Resistors_ThroughHole:Resistor_Horizontal_RM10mm" V 4030 3650 30  0001 C CNN
+F 2 "resistors:Resistor_Horizontal_RM08mm" V 4030 3650 30  0001 C CNN
 F 3 "" H 4100 3650 30  0000 C CNN
 	1    4100 3650
@@
 $EndComp
 $Comp
-L GND #PWR54
+L GND #PWR057
 U 1 1 5677F1BF
 P 4100 3900
-F 0 "#PWR54" H 4100 3650 50  0001 C CNN
+F 0 "#PWR057" H 4100 3650 50  0001 C CNN
 F 1 "GND" H 4100 3750 50  0000 C CNN
 F 2 "" H 4100 3900 60  0000 C CNN
@@
 F 0 "C15" H 6725 2350 50  0000 L CNN
 F 1 "10µF" H 6725 2150 50  0000 L CNN
-F 2 "Capacitors_ThroughHole:C_Radial_D5_L6_P2.5" H 6738 2100 30  0001 C CNN
+F 2 "Capacitors_ThroughHole:C_Radial_D5_L11_P2.5" H 6738 2100 30  0001 C CNN
 F 3 "" H 6700 2250 60  0000 C CNN
 	1    6700 2250
@@
 F 0 "R29" V 6980 2550 50  0000 C CNN
 F 1 "1k8" V 6900 2550 50  0000 C CNN
-F 2 "Resistors_ThroughHole:Resistor_Horizontal_RM10mm" V 6830 2550 30  0001 C CNN
+F 2 "resistors:Resistor_Horizontal_RM08mm" V 6830 2550 30  0001 C CNN
 F 3 "" H 6900 2550 30  0000 C CNN
 	1    6900 2550
@@
 $EndComp
 $Comp
-L GND #PWR63
+L GND #PWR058
 U 1 1 5677F1DB
 P 6900 2800
-F 0 "#PWR63" H 6900 2550 50  0001 C CNN
+F 0 "#PWR058" H 6900 2550 50  0001 C CNN
 F 1 "GND" H 6900 2650 50  0000 C CNN
 F 2 "" H 6900 2800 60  0000 C CNN
@@
 Connection ~ 6900 2250
 $Comp
-L VCC #PWR59
+L VCC #PWR059
 U 1 1 5677F1E6
 P 5500 1950
-F 0 "#PWR59" H 5500 1800 50  0001 C CNN
+F 0 "#PWR059" H 5500 1800 50  0001 C CNN
 F 1 "VCC" H 5500 2100 50  0000 C CNN
 F 2 "" H 5500 1950 60  0000 C CNN
@@
 $EndComp
 $Comp
-L VCC #PWR61
+L VCC #PWR060
 U 1 1 5677F1EC
 P 5500 3200
-F 0 "#PWR61" H 5500 3050 50  0001 C CNN
+F 0 "#PWR060" H 5500 3050 50  0001 C CNN
 F 1 "VCC" H 5500 3350 50  0000 C CNN
 F 2 "" H 5500 3200 60  0000 C CNN
@@
 $EndComp
 $Comp
-L VCC/2 #PWR58
+L VCC/2 #PWR061
 U 1 1 5677F1F2
 P 5200 3200
-F 0 "#PWR58" H 5200 3050 50  0001 C CNN
+F 0 "#PWR061" H 5200 3050 50  0001 C CNN
 F 1 "VCC/2" H 5200 3350 50  0000 C CNN
 F 2 "" H 5200 3200 60  0000 C CNN
@@
 	5200 3400 5200 3200
 $Comp
-L VCC/2 #PWR57
+L VCC/2 #PWR062
 U 1 1 5677F1FA
 P 5200 1950
-F 0 "#PWR57" H 5200 1800 50  0001 C CNN
+F 0 "#PWR062" H 5200 1800 50  0001 C CNN
 F 1 "VCC/2" H 5200 2100 50  0000 C CNN
 F 2 "" H 5200 1950 60  0000 C CNN
@@
 F 0 "R30" V 4230 2100 50  0000 C CNN
 F 1 "22k" V 4150 2100 50  0000 C CNN
-F 2 "Resistors_ThroughHole:Resistor_Horizontal_RM10mm" V 4080 2100 30  0001 C CNN
+F 2 "resistors:Resistor_Horizontal_RM08mm" V 4080 2100 30  0001 C CNN
 F 3 "" H 4150 2100 30  0000 C CNN
 	1    4150 2100

Commit message: Update footprints
Parts:
- C11: footprint Capacitors_ThroughHole:C_Rect_L7_W3.5_P5 -> Capacitors_ThroughHole:C_Rect_L7_W2.5_P5
Changed lines of the file:
@@
 F 0 "C11" H 3575 2500 50  0000 L CNN
 F 1 "100nF" H 3575 2300 50  0000 L CNN
-F 2 "Capacitors_ThroughHole:C_Rect_L7_W3.5_P5" H 3588 2250 30  0001 C CNN
+F 2 "Capacitors_ThroughHole:C_Rect_L7_W2.5_P5" H 3588 2250 30  0001 C CNN
 F 3 "" H 3550 2400 60  0000 C CNN
 	1    3550 2400
