File: schema/audio.sch (KiCad schematic (older format))
At the start: 21 parts, among them U6 TBB1458

Commit message: Component placement
Parts:
- renumbered R19 to R20, R20 to R21, R21 to R22, R22 to R23, R30 to R24, R23 to R25, R24 to R26, R25 to R27, R26 to R28, R27 to R29, R28 to R30, R29 to R31, U6 to U8
Changed lines of the file:
@@
 	2650 2100 2800 2100
 $Comp
-L R R19
+L R R20
 U 1 1 5677F0F1
 P 2950 2100
-F 0 "R19" V 3030 2100 50  0000 C CNN
+F 0 "R20" V 3030 2100 50  0000 C CNN
 F 1 "560" V 2950 2100 50  0000 C CNN
 F 2 "resistors:Resistor_Horizontal_RM08mm" V 2880 2100 30  0001 C CNN
@@
 $EndComp
 $Comp
-L GND #PWR53
+L GND #PWR053
 U 1 1 5677F0FF
 P 3150 2650
-F 0 "#PWR53" H 3150 2400 50  0001 C CNN
+F 0 "#PWR053" H 3150 2400 50  0001 C CNN
 F 1 "GND" H 3150 2500 50  0000 C CNN
 F 2 "" H 3150 2650 60  0000 C CNN
@@
 	3150 2100 3150 2250
 $Comp
-L R R20
+L R R21
 U 1 1 5677F108
 P 3350 2100
-F 0 "R20" V 3430 2100 50  0000 C CNN
+F 0 "R21" V 3430 2100 50  0000 C CNN
 F 1 "1k8" V 3350 2100 50  0000 C CNN
 F 2 "resistors:Resistor_Horizontal_RM08mm" V 3280 2100 30  0001 C CNN
@@
 $EndComp
 $Comp
-L GND #PWR54
+L GND #PWR054
 U 1 1 5677F116
 P 3550 2650
-F 0 "#PWR54" H 3550 2400 50  0001 C CNN
+F 0 "#PWR054" H 3550 2400 50  0001 C CNN
 F 1 "GND" H 3550 2500 50  0000 C CNN
 F 2 "" H 3550 2650 60  0000 C CNN
@@
 	3550 2100 3550 2250
 $Comp
-L R R21
+L R R22
 U 1 1 5677F11F
 P 3750 2100
-F 0 "R21" V 3830 2100 50  0000 C CNN
+F 0 "R22" V 3830 2100 50  0000 C CNN
 F 1 "5k6" V 3750 2100 50  0000 C CNN
 F 2 "resistors:Resistor_Horizontal_RM08mm" V 3680 2100 30  0001 C CNN
@@
 $EndComp
 $Comp
-L GND #PWR55
+L GND #PWR055
 U 1 1 5677F12D
 P 3950 2650
-F 0 "#PWR55" H 3950 2400 50  0001 C CNN
+F 0 "#PWR055" H 3950 2400 50  0001 C CNN
 F 1 "GND" H 3950 2500 50  0000 C CNN
 F 2 "" H 3950 2650 60  0000 C CNN
@@
 $EndComp
 $Comp
-L GND #PWR57
+L GND #PWR056
 U 1 1 5677F13F
 P 4400 2650
-F 0 "#PWR57" H 4400 2400 50  0001 C CNN
+F 0 "#PWR056" H 4400 2400 50  0001 C CNN
 F 1 "GND" H 4400 2500 50  0000 C CNN
 F 2 "" H 4400 2650 60  0000 C CNN
@@
 $EndComp
 $Comp
-L R R23
+L R R25
 U 1 1 5677F14E
 P 5000 2350
-F 0 "R23" V 5080 2350 50  0000 C CNN
+F 0 "R25" V 5080 2350 50  0000 C CNN
 F 1 "47k" V 5000 2350 50  0000 C CNN
 F 2 "resistors:Resistor_Horizontal_RM08mm" V 4930 2350 30  0001 C CNN
@@
 $EndComp
 $Comp
-L OP275-RESCUE-ham-relay U6
+L OP275-RESCUE-ham-relay U8
 U 1 1 5677F155
 P 5600 2250
-F 0 "U6" H 5600 2400 60  0000 L CNN
+F 0 "U8" H 5600 2400 60  0000 L CNN
 F 1 "TBB1458" H 5600 2100 60  0000 L CNN
 F 2 "Housings_DIP:DIP-8_W7.62mm" H 5600 2250 60  0001 C CNN
@@
 	5150 2350 5250 2350
 $Comp
-L R R25
+L R R27
 U 1 1 5677F15D
 P 5600 2900
-F 0 "R25" V 5680 2900 50  0000 C CNN
+F 0 "R27" V 5680 2900 50  0000 C CNN
 F 1 "220k" V 5600 2900 50  0000 C CNN
 F 2 "resistors:Resistor_Horizontal_RM08mm" V 5530 2900 30  0001 C CNN
@@
 $EndComp
 $Comp
-L GND #PWR62
+L GND #PWR057
 U 1 1 5677F164
 P 5500 2550
-F 0 "#PWR62" H 5500 2300 50  0001 C CNN
+F 0 "#PWR057" H 5500 2300 50  0001 C CNN
 F 1 "GND" H 5500 2400 50  0000 C CNN
 F 2 "" H 5500 2550 60  0000 C CNN
@@
 Connection ~ 5200 2350
 $Comp
-L R R27
+L R R29
 U 1 1 5677F16E
 P 6200 2250
-F 0 "R27" V 6280 2250 50  0000 C CNN
+F 0 "R29" V 6280 2250 50  0000 C CNN
 F 1 "1k2" V 6200 2250 50  0000 C CNN
 F 2 "resistors:Resistor_Horizontal_RM08mm" V 6130 2250 30  0001 C CNN
@@
 $EndComp
 $Comp
-L GND #PWR58
+L GND #PWR058
 U 1 1 5677F180
 P 4400 3900
-F 0 "#PWR58" H 4400 3650 50  0001 C CNN
+F 0 "#PWR058" H 4400 3650 50  0001 C CNN
 F 1 "GND" H 4400 3750 50  0000 C CNN
 F 2 "" H 4400 3900 60  0000 C CNN
@@
 $EndComp
 $Comp
-L R R24
+L R R26
 U 1 1 5677F18E
 P 5000 3600
-F 0 "R24" V 5080 3600 50  0000 C CNN
+F 0 "R26" V 5080 3600 50  0000 C CNN
 F 1 "47k" V 5000 3600 50  0000 C CNN
 F 2 "resistors:Resistor_Horizontal_RM08mm" V 4930 3600 30  0001 C CNN
@@
 	5150 3600 5250 3600
 $Comp
-L R R26
+L R R28
 U 1 1 5677F196
 P 5600 4150
-F 0 "R26" V 5680 4150 50  0000 C CNN
+F 0 "R28" V 5680 4150 50  0000 C CNN
 F 1 "220k" V 5600 4150 50  0000 C CNN
 F 2 "resistors:Resistor_Horizontal_RM08mm" V 5530 4150 30  0001 C CNN
@@
 $EndComp
 $Comp
-L GND #PWR64
+L GND #PWR059
 U 1 1 5677F19D
 P 5500 3800
-F 0 "#PWR64" H 5500 3550 50  0001 C CNN
+F 0 "#PWR059" H 5500 3550 50  0001 C CNN
 F 1 "GND" H 5500 3650 50  0000 C CNN
 F 2 "" H 5500 3800 60  0000 C CNN
@@
 Connection ~ 5200 3600
 $Comp
-L R R28
+L R R30
 U 1 1 5677F1A7
 P 6200 3500
-F 0 "R28" V 6280 3500 50  0000 C CNN
+F 0 "R30" V 6280 3500 50  0000 C CNN
 F 1 "1k2" V 6200 3500 50  0000 C CNN
 F 2 "resistors:Resistor_Horizontal_RM08mm" V 6130 3500 30  0001 C CNN
@@
 Connection ~ 6000 3500
 $Comp
-L OP275-RESCUE-ham-relay U6
+L OP275-RESCUE-ham-relay U8
 U 2 1 5677F1B1
 P 5600 3500
-F 0 "U6" H 5600 3650 60  0000 L CNN
+F 0 "U8" H 5600 3650 60  0000 L CNN
 F 1 "TBB1458" H 5600 3350 60  0000 L CNN
 F 2 "Housings_DIP:DIP-8_W7.62mm" H 5600 3500 60  0001 C CNN
@@
 $EndComp
 $Comp
-L R R22
+L R R23
 U 1 1 5677F1B8
 P 4100 3650
-F 0 "R22" V 4180 3650 50  0000 C CNN
+F 0 "R23" V 4180 3650 50  0000 C CNN
 F 1 "1k8" V 4100 3650 50  0000 C CNN
 F 2 "resistors:Resistor_Horizontal_RM08mm" V 4030 3650 30  0001 C CNN
@@
 $EndComp
 $Comp
-L GND #PWR56
+L GND #PWR060
 U 1 1 5677F1BF
 P 4100 3900
-F 0 "#PWR56" H 4100 3650 50  0001 C CNN
+F 0 "#PWR060" H 4100 3650 50  0001 C CNN
 F 1 "GND" H 4100 3750 50  0000 C CNN
 F 2 "" H 4100 3900 60  0000 C CNN
@@
 $EndComp
 $Comp
-L R R29
+L R R31
 U 1 1 5677F1D4
 P 6900 2550
-F 0 "R29" V 6980 2550 50  0000 C CNN
+F 0 "R31" V 6980 2550 50  0000 C CNN
 F 1 "1k8" V 6900 2550 50  0000 C CNN
 F 2 "resistors:Resistor_Horizontal_RM08mm" V 6830 2550 30  0001 C CNN
@@
 $EndComp
 $Comp
-L GND #PWR65
+L GND #PWR061
 U 1 1 5677F1DB
 P 6900 2800
-F 0 "#PWR65" H 6900 2550 50  0001 C CNN
+F 0 "#PWR061" H 6900 2550 50  0001 C CNN
 F 1 "GND" H 6900 2650 50  0000 C CNN
 F 2 "" H 6900 2800 60  0000 C CNN
@@
 Connection ~ 6900 2250
 $Comp
-L VCC #PWR61
+L VCC #PWR062
 U 1 1 5677F1E6
 P 5500 1950
-F 0 "#PWR61" H 5500 1800 50  0001 C CNN
+F 0 "#PWR062" H 5500 1800 50  0001 C CNN
 F 1 "VCC" H 5500 2100 50  0000 C CNN
 F 2 "" H 5500 1950 60  0000 C CNN
@@
 $EndComp
 $Comp
-L VCC #PWR63
+L VCC #PWR063
 U 1 1 5677F1EC
 P 5500 3200
-F 0 "#PWR63" H 5500 3050 50  0001 C CNN
+F 0 "#PWR063" H 5500 3050 50  0001 C CNN
 F 1 "VCC" H 5500 3350 50  0000 C CNN
 F 2 "" H 5500 3200 60  0000 C CNN
@@
 $EndComp
 $Comp
-L VCC/2 #PWR60
+L VCC/2 #PWR064
 U 1 1 5677F1F2
 P 5200 3200
-F 0 "#PWR60" H 5200 3050 50  0001 C CNN
+F 0 "#PWR064" H 5200 3050 50  0001 C CNN
 F 1 "VCC/2" H 5200 3350 50  0000 C CNN
 F 2 "" H 5200 3200 60  0000 C CNN
@@
 	5200 3400 5200 3200
 $Comp
-L VCC/2 #PWR59
+L VCC/2 #PWR065
 U 1 1 5677F1FA
 P 5200 1950
-F 0 "#PWR59" H 5200 1800 50  0001 C CNN
+F 0 "#PWR065" H 5200 1800 50  0001 C CNN
 F 1 "VCC/2" H 5200 2100 50  0000 C CNN
 F 2 "" H 5200 1950 60  0000 C CNN
@@
 TONE
 $Comp
-L R R30
+L R R24
 U 1 1 567C5134
 P 4150 2100
-F 0 "R30" V 4230 2100 50  0000 C CNN
+F 0 "R24" V 4230 2100 50  0000 C CNN
 F 1 "22k" V 4150 2100 50  0000 C CNN
 F 2 "resistors:Resistor_Horizontal_RM08mm" V 4080 2100 30  0001 C CNN

Commit message: Start fixing schematics
Parts:
- R27: value 220k -> 680k
- R28: value 220k -> 330k
- RV1, RV2: symbol POT -> POT-RESCUE-ham-relay
Changed lines of the file:
@@
 Sheet 2 2
 Title "Logique relais"
-Date "2016-02-14"
-Rev "6"
+Date "2016-04-08"
+Rev "7"
 Comp ""
 Comment1 ""
@@
 Connection ~ 3550 2100
 $Comp
-L POT RV1
+L POT-RESCUE-ham-relay RV1
 U 1 1 5677F138
 P 4400 2350
+AR Path="/5677F138" Ref="RV1"  Part="1"
+AR Path="/5677D530/5677F138" Ref="RV1"  Part="1"
 F 0 "RV1" H 4400 2250 50  0000 C CNN
 F 1 "10k" H 4400 2350 50  0000 C CNN
@@
 P 5600 2900
 F 0 "R27" V 5680 2900 50  0000 C CNN
-F 1 "220k" V 5600 2900 50  0000 C CNN
+F 1 "680k" V 5600 2900 50  0000 C CNN
 F 2 "resistors:Resistor_Horizontal_RM08mm" V 5530 2900 30  0001 C CNN
 F 3 "" H 5600 2900 30  0000 C CNN
@@
 	3950 3350 4400 3350
 $Comp
-L POT RV2
+L POT-RESCUE-ham-relay RV2
 U 1 1 5677F179
 P 4400 3600
+AR Path="/5677F179" Ref="RV2"  Part="1"
+AR Path="/5677D530/5677F179" Ref="RV2"  Part="1"
 F 0 "RV2" H 4400 3500 50  0000 C CNN
 F 1 "1k" H 4400 3600 50  0000 C CNN
@@
 P 5600 4150
 F 0 "R28" V 5680 4150 50  0000 C CNN
-F 1 "220k" V 5600 4150 50  0000 C CNN
+F 1 "330k" V 5600 4150 50  0000 C CNN
 F 2 "resistors:Resistor_Horizontal_RM08mm" V 5530 4150 30  0001 C CNN
 F 3 "" H 5600 4150 30  0000 C CNN
